Commit message: update jaco urdf

File: robots/jaco_description/urdf/jaco_arm.urdf (robot description, URDF)
Before this commit: robot jaco, 7 links, 6 joints
Links:
- added link base_link
- added link jaco_large_ring_cover_1, mass 0.001; collision mesh filename=package://jaco_description/meshes/jaco_large_ring_cover.stl scale=0.0254 0.0254 0.0254; visual mesh filename=package://jaco_description/meshes/jaco_large_ring_cover.min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 scale=0.0254 0.0254 0.0254
- added link jaco_large_ring_cover_2, mass 0.001; collision mesh filename=package://jaco_description/meshes/jaco_large_ring_cover.stl scale=0.0254 0.0254 0.0254; visual mesh filename=package://jaco_description/meshes/jaco_large_ring_cover.min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 scale=0.0254 0.0254 0.0254
- added link jaco_large_ring_cover_3, mass 0.001; collision mesh filename=package://jaco_description/meshes/jaco_large_ring_cover.stl scale=0.0254 0.0254 0.0254; visual mesh filename=package://jaco_description/meshes/jaco_large_ring_cover.min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 scale=0.0254 0.0254 0.0254
- added link jaco_link_finger_1, mass 0.25; collision mesh filename=package://jaco_description/meshes/jaco_link_finger.stl scale=0.0254 0.0254 0.0254; visual mesh filename=package://jaco_description/meshes/jaco_link_finger.min.dae scale=0.0254 0.0254 0.0254
- added link jaco_link_finger_2, mass 0.25; collision mesh filename=package://jaco_description/meshes/jaco_link_finger.stl scale=0.0254 0.0254 0.0254; visual mesh filename=package://jaco_description/meshes/jaco_link_finger.min.dae scale=0.0254 0.0254 0.0254
- added link jaco_link_finger_3, mass 0.25; collision mesh filename=package://jaco_description/meshes/jaco_link_finger.stl scale=0.0254 0.0254 0.0254; visual mesh filename=package://jaco_description/meshes/jaco_link_finger.min.dae scale=0.0254 0.0254 0.0254
- added link jaco_link_finger_tip_1, mass 0.25; collision mesh filename=package://jaco_description/meshes/jaco_link_finger_tip.stl scale=0.0254 0.0254 0.0254; visual mesh filename=package://jaco_description/meshes/jaco_link_finger_tip.min.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 scale=0.0254 0.0254 0.0254
- added link jaco_link_finger_tip_2, mass 0.25; collision mesh filename=package://jaco_description/meshes/jaco_link_finger_tip.stl scale=0.0254 0.0254 0.0254; visual mesh filename=package://jaco_description/meshes/jaco_link_finger_tip.min.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 scale=0.0254 0.0254 0.0254
- added link jaco_link_finger_tip_3, mass 0.25; collision mesh filename=package://jaco_description/meshes/jaco_link_finger_tip.stl scale=0.0254 0.0254 0.0254; visual mesh filename=package://jaco_description/meshes/jaco_link_finger_tip.min.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 scale=0.0254 0.0254 0.0254
- added link jaco_small_ring_cover_1, mass 0.001; collision mesh filename=package://jaco_description/meshes/jaco_small_ring_cover.stl scale=0.0254 0.0254 0.0254; visual mesh filename=package://jaco_description/meshes/jaco_small_ring_cover.min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 scale=0.0254 0.0254 0.0254
- added link jaco_small_ring_cover_2, mass 0.001; collision mesh filename=package://jaco_description/meshes/jaco_small_ring_cover.stl scale=0.0254 0.0254 0.0254; visual mesh filename=package://jaco_description/meshes/jaco_small_ring_cover.min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 scale=0.0254 0.0254 0.0254
- added link jaco_small_ring_cover_3, mass 0.001; collision mesh filename=package://jaco_description/meshes/jaco_small_ring_cover.stl scale=0.0254 0.0254 0.0254; visual mesh filename=package://jaco_description/meshes/jaco_small_ring_cover.min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 scale=0.0254 0.0254 0.0254
Joints:
- added joint jaco_joint_base: type fixed, parent base_link, child jaco_link_base, origin xyz=0 0 0 rpy=0 0 0, axis 0 0 0, limit lower=-6.283185307179586 upper=6.283185307179586 effort=30 velocity=5
- added joint jaco_joint_finger_1: type revolute, parent jaco_link_hand, child jaco_link_finger_1, origin xyz=-0.032578 0.0033 -0.12131 rpy=-1.7983 1.117 3.1416, axis 0 0 1, limit lower=0 upper=0.6981317007977318 effort=30 velocity=5
- added joint jaco_joint_finger_2: type revolute, parent jaco_link_hand, child jaco_link_finger_2, origin xyz=0.027788 0.0206 -0.12131 rpy=-1.5161 1.1459 0.23978, axis 0 0 1, limit lower=0 upper=0.6981317007977318 effort=30 velocity=5
- added joint jaco_joint_finger_3: type revolute, parent jaco_link_hand, child jaco_link_finger_3, origin xyz=0.027788 -0.0206 -0.12131 rpy=-1.6222 1.117 -0.23615, axis 0 0 1, limit lower=0 upper=0.6981317007977318 effort=30 velocity=5
- added joint jaco_joint_finger_tip_1: type revolute, parent jaco_link_finger_1, child jaco_link_finger_tip_1, origin xyz=0.044094 -0.0029 0 rpy=0 0 0, axis 0 0 1, limit lower=0 upper=0.6981317007977318 effort=30 velocity=5
- added joint jaco_joint_finger_tip_2: type revolute, parent jaco_link_finger_2, child jaco_link_finger_tip_2, origin xyz=0.044094 -0.0029 0 rpy=0 0 0, axis 0 0 1, limit lower=0 upper=0.6981317007977318 effort=30 velocity=5
- added joint jaco_joint_finger_tip_3: type revolute, parent jaco_link_finger_3, child jaco_link_finger_tip_3, origin xyz=0.044094 -0.0029 0 rpy=0 0 0, axis 0 0 1, limit lower=0 upper=0.6981317007977318 effort=30 velocity=5
- added joint jaco_large_ring_cover_1_joint: type fixed, parent jaco_link_base, child jaco_large_ring_cover_1, origin xyz=0 0 0.1535 rpy=3.141592653589793 0 0, axis 0 0 1, limit lower=-6.283185307179586 upper=6.283185307179586 effort=30 velocity=5
- added joint jaco_large_ring_cover_2_joint: type fixed, parent jaco_link_1, child jaco_large_ring_cover_2, origin xyz=0 0 -0.1185 rpy=-1.5707963267948966 -1.5707963267948966 0, axis 0 0 1, limit lower=0 upper=6.283185307179586 effort=30 velocity=5
- added joint jaco_large_ring_cover_3_joint: type fixed, parent jaco_link_2, child jaco_large_ring_cover_3, origin xyz=0.41 0 0 rpy=3.141592653589793 0 3.141592653589793, axis 0 0 1, limit lower=0 upper=6.283185307179586 effort=30 velocity=5
- added joint jaco_large_ring_cover_4_joint: type fixed, parent jaco_link_3, child jaco_small_ring_cover_1, origin xyz=0.207 0 -0.01125 rpy=0 -1.5707963267948966 0, axis 0 0 1, limit lower=-6.283185307179586 upper=6.283185307179586 effort=30 velocity=5
- added joint jaco_large_ring_cover_5_joint: type fixed, parent jaco_link_4, child jaco_small_ring_cover_2, origin xyz=0.0343 0 -0.06588 rpy=0 0.9599310885968813 3.141592653589793, axis 0 0 1, limit lower=-6.283185307179586 upper=6.283185307179586 effort=30 velocity=5
- added joint jaco_large_ring_cover_6_joint: type fixed, parent jaco_link_5, child jaco_small_ring_cover_3, origin xyz=0.0343 0 -0.06588 rpy=0 0.9599310885968813 3.141592653589793, axis 0 0 1, limit lower=-6.283185307179586 upper=6.283185307179586 effort=30 velocity=5
